Commit message: Release/Flexiv ROS 2 Humble v1.9 (#90)

File: flexiv_moveit_config/srdf/grav.srdf.xacro (robot description, xacro)
@@ -4,5 +4,5 @@
         <!-- Prefix defaults to 'arm_prefix_robot_sn' -->
         <xacro:property name="prefix" value="${arm_prefix + robot_sn + '_'}" />
-        <group name="grav_gripper">
+        <group name="${prefix}grav_gripper">
             <joint name="${prefix}gripper_base_joint" />
             <joint name="${prefix}open_fingers_tcp_joint" />
@@ -26,12 +26,12 @@
         <passive_joint name="${prefix}right_inner_knuckle_joint" />
         <passive_joint name="${prefix}right_inner_finger_joint" />
-        <group_state name="open" group="grav_gripper">
+        <group_state name="${prefix}open" group="${prefix}grav_gripper">
             <joint name="${prefix}finger_width_joint" value="0.1" />
         </group_state>
-        <group_state name="closed" group="grav_gripper">
+        <group_state name="${prefix}closed" group="${prefix}grav_gripper">
             <joint name="${prefix}finger_width_joint" value="0.0" />
         </group_state>
-        <end_effector name="grav_gripper" parent_link="${prefix}flange"
-            group="grav_gripper" parent_group="rizon_arm" />
+        <end_effector name="${prefix}grav_gripper" parent_link="${prefix}flange"
+            group="${prefix}grav_gripper" parent_group="${prefix}arm" />
         <disable_collisions link1="${prefix}grav_base_link" link2="${prefix}grav_tcp" reason="Never" />
         <disable_collisions link1="${prefix}grav_base_link" link2="${prefix}closed_fingers_tcp"

File: flexiv_moveit_config/srdf/rizon_macro.srdf.xacro (robot description, xacro)
@@ -1,11 +1,11 @@
 <?xml version="1.0" encoding="UTF-8"?>
 <robot xmlns:xacro="http://www.ros.org/wiki/xacro">
-    <xacro:macro name="rizon_srdf" params="arm_prefix robot_sn load_mounted_ft_sensor">
+    <xacro:macro name="rizon_srdf" params="arm_prefix robot_sn load_mounted_ft_sensor use_virtual_joint:=true">
         <!-- Prefix defaults to 'arm_prefix_robot_sn' -->
         <xacro:property name="prefix" value="${arm_prefix + robot_sn + '_'}" />
-        <group name="rizon_arm">
+        <group name="${prefix}arm">
             <chain base_link="${prefix}base_link" tip_link="${prefix}flange" />
         </group>
-        <group_state name="${prefix}home" group="rizon_arm">
+        <group_state name="${prefix}home" group="${prefix}arm">
             <joint name="${prefix}joint1" value="0" />
             <joint name="${prefix}joint2" value="${-2*pi/9}" />
@@ -16,6 +16,8 @@
             <joint name="${prefix}joint7" value="0" />
         </group_state>
-        <virtual_joint name="virtual_joint" type="fixed" parent_frame="world"
-            child_link="${prefix}base_link" />
+        <xacro:if value="${use_virtual_joint}">
+            <virtual_joint name="virtual_joint" type="fixed" parent_frame="world"
+                child_link="${prefix}base_link" />
+        </xacro:if>
         <disable_collisions link1="${prefix}base_link" link2="${prefix}link1" reason="Adjacent" />
         <disable_collisions link1="${prefix}base_link" link2="${prefix}link2" reason="Never" />
@@ -40,16 +42,10 @@
         <xacro:if value="${load_mounted_ft_sensor}">
             <!-- Disable collisions for FT sensor fixed-link chain -->
-            <disable_collisions link1="${prefix}link7" link2="${prefix}wrist-sensor.base_link"
-                reason="Adjacent" />
-            <disable_collisions link1="${prefix}wrist-sensor.base_link"
-                link2="${prefix}wrist-sensor.proximal_link" reason="Adjacent" />
-            <disable_collisions link1="${prefix}wrist-sensor.proximal_link"
-                link2="${prefix}wrist-sensor.distal_link" reason="Adjacent" />
-            <disable_collisions link1="${prefix}wrist-sensor.distal_link" link2="${prefix}flange"
-                reason="Adjacent" />
-            <disable_collisions link1="${prefix}link7" link2="${prefix}wrist-sensor.proximal_link"
-                reason="Adjacent" />
-            <disable_collisions link1="${prefix}link7" link2="${prefix}wrist-sensor.distal_link"
-                reason="Adjacent" />
+            <disable_collisions link1="${prefix}link7" link2="${prefix}wrist-sensor.base_link" reason="Adjacent" />
+            <disable_collisions link1="${prefix}wrist-sensor.base_link" link2="${prefix}wrist-sensor.proximal_link" reason="Adjacent" />
+            <disable_collisions link1="${prefix}wrist-sensor.proximal_link" link2="${prefix}wrist-sensor.distal_link" reason="Adjacent" />
+            <disable_collisions link1="${prefix}wrist-sensor.distal_link" link2="${prefix}flange" reason="Adjacent" />
+            <disable_collisions link1="${prefix}link7" link2="${prefix}wrist-sensor.proximal_link" reason="Adjacent" />
+            <disable_collisions link1="${prefix}link7" link2="${prefix}wrist-sensor.distal_link" reason="Adjacent" />
         </xacro:if>
     </xacro:macro>
