Commit message: Task/Adapt to consolidated flexiv_description (humble-v1.9.3) (#114)

File: flexiv_moveit_config/srdf/aico1.srdf.xacro (robot description, xacro)
@@ -2,19 +2,23 @@
 <robot xmlns:xacro="http://wiki.ros.org/xacro" name="aico1">
     <!-- parameters -->
-    <xacro:arg name="external_axis_type" default="aico1_4_v1" />
+    <xacro:arg name="robot_type" default="AICO1-4-V1" />
+    <!-- Axis macro/link names are the robot type lowercased with dashes as
+         underscores, e.g. AICO2-10-V1 -> aico2_10_v1. -->
+    <xacro:property name="axis_name"
+      value="${'$(arg robot_type)'.lower().replace('-', '_')}" />
     <xacro:arg name="external_axis_prefix" default="" />
-    <xacro:arg name="arm_prefix" default="" />
     <xacro:arg name="robot_sn" default="" />
     <xacro:arg name="load_gripper" default="false" />
     <xacro:arg name="load_mounted_ft_sensor" default="false" />
     <xacro:include filename="$(find flexiv_moveit_config)/srdf/rizon_macro.srdf.xacro" />
+    <!-- Prefixes -->
+    <xacro:compute_prefix robot_sn="$(arg robot_sn)" />
+    <xacro:property name="prefix" value="${computed_prefix}" lazy_eval="false" />
     <!-- Arm -->
-    <xacro:rizon_srdf arm_prefix="$(arg arm_prefix)" robot_sn="$(arg robot_sn)"
+    <xacro:rizon_srdf prefix="${prefix}"
         load_mounted_ft_sensor="$(arg load_mounted_ft_sensor)" use_virtual_joint="false" />
-    <!-- Prefixes -->
-    <xacro:property name="prefix" value="$(arg arm_prefix)$(arg robot_sn)_" />
     <xacro:property name="external_axis_prefix" value="$(arg external_axis_prefix)" />
     <!-- Virtual Joint and Platform Group -->
-    <xacro:if value="${'$(arg external_axis_type)' == 'aico1_4_v1'}">
+    <xacro:if value="${axis_name == 'aico1_4_v1'}">
         <virtual_joint name="virtual_joint" type="fixed" parent_frame="world"
             child_link="${external_axis_prefix}aico1_4_v1_base_link" />
@@ -23,5 +27,5 @@
         </group>
     </xacro:if>
-    <xacro:if value="${'$(arg external_axis_type)' == 'aico1_4_v2'}">
+    <xacro:if value="${axis_name == 'aico1_4_v2'}">
         <virtual_joint name="virtual_joint" type="fixed" parent_frame="world"
             child_link="${external_axis_prefix}aico1_4_v2_base_link" />
@@ -31,5 +35,5 @@
     </xacro:if>
     <!-- Platform Collisions -->
-    <xacro:if value="${'$(arg external_axis_type)' == 'aico1_4_v1'}">
+    <xacro:if value="${axis_name == 'aico1_4_v1'}">
         <disable_collisions link1="${prefix}base_link" link2="${external_axis_prefix}aico1_4_v1_link2" reason="Adjacent" />
         <disable_collisions link1="${prefix}base_link" link2="${external_axis_prefix}aico1_4_v1_link1" reason="Never" />
@@ -42,5 +46,5 @@
         <disable_collisions link1="${external_axis_prefix}aico1_4_v1_link1" link2="${external_axis_prefix}aico1_4_v1_link2" reason="Adjacent" />
     </xacro:if>
-    <xacro:if value="${'$(arg external_axis_type)' == 'aico1_4_v2'}">
+    <xacro:if value="${axis_name == 'aico1_4_v2'}">
         <disable_collisions link1="${prefix}base_link" link2="${external_axis_prefix}aico1_4_v2_link1" reason="Adjacent" />
         <disable_collisions link1="${prefix}base_link" link2="${external_axis_prefix}aico1_4_v2_base_link" reason="Never" />
@@ -59,5 +63,5 @@
     <xacro:if value="$(arg load_gripper)">
         <xacro:include filename="$(find flexiv_moveit_config)/srdf/grav.srdf.xacro" />
-        <xacro:grav_srdf arm_prefix="$(arg arm_prefix)" robot_sn="$(arg robot_sn)"
+        <xacro:grav_srdf prefix="${prefix}"
             load_mounted_ft_sensor="$(arg load_mounted_ft_sensor)" />
     </xacro:if>

File: flexiv_moveit_config/srdf/aico2.srdf.xacro (robot description, xacro)
@@ -2,5 +2,9 @@
 <robot xmlns:xacro="http://wiki.ros.org/xacro" name="aico2">
     <!-- parameters -->
-    <xacro:arg name="external_axis_type" default="aico2_4_v1" />
+    <xacro:arg name="robot_type" default="AICO2-4-V1" />
+    <!-- Axis macro/link names are the robot type lowercased with dashes as
+         underscores, e.g. AICO2-10-V1 -> aico2_10_v1. -->
+    <xacro:property name="axis_name"
+      value="${'$(arg robot_type)'.lower().replace('-', '_')}" />
     <xacro:arg name="external_axis_prefix" default="" />
     <xacro:arg name="robot_sn_left" default="" />
@@ -10,19 +14,21 @@
     <xacro:arg name="load_mounted_ft_sensor_left" default="false" />
     <xacro:arg name="load_mounted_ft_sensor_right" default="false" />
-    <xacro:arg name="arm_prefix_left" default="left_" />
-    <xacro:arg name="arm_prefix_right" default="right_" />
+    <xacro:arg name="arm_prefix_left" default="left" />
+    <xacro:arg name="arm_prefix_right" default="right" />
     <xacro:include filename="$(find flexiv_moveit_config)/srdf/rizon_macro.srdf.xacro" />
+    <!-- Prefixes. lazy_eval is off so each capture resolves before the next call. -->
+    <xacro:compute_prefix side="$(arg arm_prefix_left)" robot_sn="$(arg robot_sn_left)" />
+    <xacro:property name="prefix_left" value="${computed_prefix}" lazy_eval="false" />
+    <xacro:compute_prefix side="$(arg arm_prefix_right)" robot_sn="$(arg robot_sn_right)" />
+    <xacro:property name="prefix_right" value="${computed_prefix}" lazy_eval="false" />
+    <xacro:property name="external_axis_prefix" value="$(arg external_axis_prefix)" />
     <!-- Left Arm -->
-    <xacro:rizon_srdf arm_prefix="$(arg arm_prefix_left)" robot_sn="$(arg robot_sn_left)"
+    <xacro:rizon_srdf prefix="${prefix_left}"
         load_mounted_ft_sensor="$(arg load_mounted_ft_sensor_left)" use_virtual_joint="false" />
     <!-- Right Arm -->
-    <xacro:rizon_srdf arm_prefix="$(arg arm_prefix_right)" robot_sn="$(arg robot_sn_right)"
+    <xacro:rizon_srdf prefix="${prefix_right}"
         load_mounted_ft_sensor="$(arg load_mounted_ft_sensor_right)" use_virtual_joint="false" />
-    <!-- Prefixes -->
-    <xacro:property name="prefix_left" value="$(arg arm_prefix_left)$(arg robot_sn_left)_" />
-    <xacro:property name="prefix_right" value="$(arg arm_prefix_right)$(arg robot_sn_right)_" />
-    <xacro:property name="external_axis_prefix" value="$(arg external_axis_prefix)" />
     <!-- Virtual Joint and External Axis Group -->
-    <xacro:if value="${'$(arg external_axis_type)' == 'aico2_4_v1'}">
+    <xacro:if value="${axis_name == 'aico2_4_v1'}">
         <virtual_joint name="virtual_joint" type="fixed" parent_frame="world"
             child_link="${external_axis_prefix}aico2_4_v1_base_link" />
@@ -31,5 +37,5 @@
         </group>
     </xacro:if>
-    <xacro:if value="${'$(arg external_axis_type)' == 'aico2_4_v2'}">
+    <xacro:if value="${axis_name == 'aico2_4_v2'}">
         <virtual_joint name="virtual_joint" type="fixed" parent_frame="world"
             child_link="${external_axis_prefix}aico2_4_v2_base_link" />
@@ -38,5 +44,5 @@
         </group>
     </xacro:if>
-    <xacro:if value="${'$(arg external_axis_type)' == 'aico2_10_v1'}">
+    <xacro:if value="${axis_name == 'aico2_10_v1'}">
         <virtual_joint name="virtual_joint" type="fixed" parent_frame="world"
             child_link="${external_axis_prefix}aico2_10_v1_base_link" />
@@ -46,5 +52,5 @@
     </xacro:if>
     <!-- External Axis Collisions -->
-    <xacro:if value="${'$(arg external_axis_type)' == 'aico2_4_v1'}">
+    <xacro:if value="${axis_name == 'aico2_4_v1'}">
         <!-- Left Arm -->
         <disable_collisions link1="${prefix_left}base_link" link2="${external_axis_prefix}aico2_4_v1_link2" reason="Adjacent" />
@@ -69,5 +75,5 @@
         <disable_collisions link1="${external_axis_prefix}aico2_4_v1_link1" link2="${external_axis_prefix}aico2_4_v1_link2" reason="Adjacent" />
     </xacro:if>
-    <xacro:if value="${'$(arg external_axis_type)' == 'aico2_4_v2'}">
+    <xacro:if value="${axis_name == 'aico2_4_v2'}">
         <!-- Left Arm -->
         <disable_collisions link1="${prefix_left}base_link" link2="${external_axis_prefix}aico2_4_v2_link2" reason="Adjacent" />
@@ -92,5 +98,5 @@
         <disable_collisions link1="${external_axis_prefix}aico2_4_v2_link1" link2="${external_axis_prefix}aico2_4_v2_link2" reason="Adjacent" />
     </xacro:if>
-    <xacro:if value="${'$(arg external_axis_type)' == 'aico2_10_v1'}">
+    <xacro:if value="${axis_name == 'aico2_10_v1'}">
         <!-- Left Arm -->
         <disable_collisions link1="${prefix_left}base_link" link2="${external_axis_prefix}aico2_10_v1_link2" reason="Adjacent" />
@@ -118,10 +124,10 @@
     <xacro:if value="$(arg load_gripper_left)">
         <xacro:include filename="$(find flexiv_moveit_config)/srdf/grav.srdf.xacro" />
-        <xacro:grav_srdf arm_prefix="$(arg prefix_left)" robot_sn="$(arg robot_sn_left)"
+        <xacro:grav_srdf prefix="${prefix_left}"
             load_mounted_ft_sensor="$(arg load_mounted_ft_sensor_left)" />
     </xacro:if>
     <xacro:if value="$(arg load_gripper_right)">
         <xacro:include filename="$(find flexiv_moveit_config)/srdf/grav.srdf.xacro" />
-        <xacro:grav_srdf arm_prefix="$(arg prefix_right)" robot_sn="$(arg robot_sn_right)"
+        <xacro:grav_srdf prefix="${prefix_right}"
             load_mounted_ft_sensor="$(arg load_mounted_ft_sensor_right)" />
     </xacro:if>

File: flexiv_moveit_config/srdf/grav.srdf.xacro (robot description, xacro)
@@ -1,7 +1,6 @@
 <?xml version="1.0" encoding="UTF-8"?>
 <robot xmlns:xacro="http://www.ros.org/wiki/xacro">
-    <xacro:macro name="grav_srdf" params="arm_prefix robot_sn load_mounted_ft_sensor">
-        <!-- Prefix defaults to 'arm_prefix_robot_sn' -->
-        <xacro:property name="prefix" value="${arm_prefix + robot_sn + '_'}" />
+    <!-- 'prefix' is the fully-formed prefix, see compute_prefix in rizon_macro.srdf.xacro. -->
+    <xacro:macro name="grav_srdf" params="prefix load_mounted_ft_sensor">
         <group name="${prefix}grav_gripper">
             <joint name="${prefix}gripper_base_joint" />

File: flexiv_moveit_config/srdf/rizon.srdf.xacro (robot description, xacro)
@@ -1,17 +1,18 @@
 <?xml version="1.0" encoding="UTF-8"?>
-<robot xmlns:xacro="http://wiki.ros.org/xacro" name="$(arg rizon_type)">
+<robot xmlns:xacro="http://wiki.ros.org/xacro" name="$(arg robot_type)">
     <!-- parameters -->
-    <xacro:arg name="rizon_type" default="Rizon4" />
-    <xacro:arg name="arm_prefix" default="" />
+    <xacro:arg name="robot_type" default="Rizon4" />
     <xacro:arg name="robot_sn" default="" />
     <xacro:arg name="load_gripper" default="false" />
     <xacro:arg name="load_mounted_ft_sensor" default="false" />
     <xacro:include filename="$(find flexiv_moveit_config)/srdf/rizon_macro.srdf.xacro" />
-    <xacro:rizon_srdf arm_prefix="$(arg arm_prefix)" robot_sn="$(arg robot_sn)"
+    <xacro:compute_prefix robot_sn="$(arg robot_sn)" />
+    <xacro:property name="prefix" value="${computed_prefix}" lazy_eval="false" />
+    <xacro:rizon_srdf prefix="${prefix}"
         load_mounted_ft_sensor="$(arg load_mounted_ft_sensor)" />
     <!-- Load gripper -->
     <xacro:if value="$(arg load_gripper)">
         <xacro:include filename="$(find flexiv_moveit_config)/srdf/grav.srdf.xacro" />
-        <xacro:grav_srdf arm_prefix="$(arg arm_prefix)" robot_sn="$(arg robot_sn)"
+        <xacro:grav_srdf prefix="${prefix}"
             load_mounted_ft_sensor="$(arg load_mounted_ft_sensor)" />
     </xacro:if>

File: flexiv_moveit_config/srdf/rizon_dual.srdf.xacro (robot description, xacro)
@@ -8,16 +8,19 @@
     <xacro:arg name="load_mounted_ft_sensor_left" default="false" />
     <xacro:arg name="load_mounted_ft_sensor_right" default="false" />
-    <xacro:arg name="prefix_left" default="left_" />
-    <xacro:arg name="prefix_right" default="right_" />
+    <!-- Side names carry no trailing underscore; compute_prefix inserts the separator. -->
+    <xacro:arg name="prefix_left" default="left" />
+    <xacro:arg name="prefix_right" default="right" />
     <xacro:include filename="$(find flexiv_moveit_config)/srdf/rizon_macro.srdf.xacro" />
+    <!-- Arm Prefixes. lazy_eval is off so each capture resolves before the next call. -->
+    <xacro:compute_prefix side="$(arg prefix_left)" robot_sn="$(arg robot_sn_left)" />
+    <xacro:property name="left_arm_prefix" value="${computed_prefix}" lazy_eval="false" />
+    <xacro:compute_prefix side="$(arg prefix_right)" robot_sn="$(arg robot_sn_right)" />
+    <xacro:property name="right_arm_prefix" value="${computed_prefix}" lazy_eval="false" />
     <!-- Left Arm -->
-    <xacro:rizon_srdf arm_prefix="$(arg prefix_left)" robot_sn="$(arg robot_sn_left)"
+    <xacro:rizon_srdf prefix="${left_arm_prefix}"
         load_mounted_ft_sensor="$(arg load_mounted_ft_sensor_left)" />
     <!-- Right Arm -->
-    <xacro:rizon_srdf arm_prefix="$(arg prefix_right)" robot_sn="$(arg robot_sn_right)"
+    <xacro:rizon_srdf prefix="${right_arm_prefix}"
         load_mounted_ft_sensor="$(arg load_mounted_ft_sensor_right)" />
-    <!-- Arm Prefixes -->
-    <xacro:property name="left_arm_prefix" value="$(arg prefix_left)$(arg robot_sn_left)_" />
-    <xacro:property name="right_arm_prefix" value="$(arg prefix_right)$(arg robot_sn_right)_" />
     <!-- Left and Right Arms Collisions -->
     <disable_collisions link1="${left_arm_prefix}base_link" link2="${right_arm_prefix}base_link" reason="Never" />
@@ -26,10 +29,10 @@
     <xacro:if value="$(arg load_gripper_left)">
         <xacro:include filename="$(find flexiv_moveit_config)/srdf/grav.srdf.xacro" />
-        <xacro:grav_srdf arm_prefix="$(arg prefix_left)" robot_sn="$(arg robot_sn_left)"
+        <xacro:grav_srdf prefix="${left_arm_prefix}"
             load_mounted_ft_sensor="$(arg load_mounted_ft_sensor_left)" />
     </xacro:if>
     <xacro:if value="$(arg load_gripper_right)">
         <xacro:include filename="$(find flexiv_moveit_config)/srdf/grav.srdf.xacro" />
-        <xacro:grav_srdf arm_prefix="$(arg prefix_right)" robot_sn="$(arg robot_sn_right)"
+        <xacro:grav_srdf prefix="${right_arm_prefix}"
             load_mounted_ft_sensor="$(arg load_mounted_ft_sensor_right)" />
     </xacro:if>

File: flexiv_moveit_config/srdf/rizon_macro.srdf.xacro (robot description, xacro)
@@ -1,7 +1,21 @@
 <?xml version="1.0" encoding="UTF-8"?>
 <robot xmlns:xacro="http://www.ros.org/wiki/xacro">
-    <xacro:macro name="rizon_srdf" params="arm_prefix robot_sn load_mounted_ft_sensor use_virtual_joint:=true">
-        <!-- Prefix defaults to 'arm_prefix_robot_sn' -->
-        <xacro:property name="prefix" value="${arm_prefix + robot_sn + '_'}" />
+    <!--
+        Build a link/joint name prefix from a side name and a serial number, and expose
+        it to the caller as 'computed_prefix'.
+        Mirrors compute_arm_prefix in flexiv_description's flexiv_common.xacro and must
+        stay in step with it: the separating underscore only appears when the part it
+        separates is non-empty. Concatenating unconditionally yields 'left__base_link'
+        for an empty robot_sn where the URDF creates 'left_base_link'.
+        side:     'left', 'right' or '' (no trailing underscore)
+        robot_sn: robot serial number, may be empty
+    -->
+    <xacro:macro name="compute_prefix" params="side:='' robot_sn:=''">
+        <xacro:property name="computed_prefix"
+            value="${(side + '_' + robot_sn + '_') if side != '' and robot_sn != '' else (side + robot_sn + '_') if (side + robot_sn) != '' else ''}"
+            scope="parent" />
+    </xacro:macro>
+    <!-- 'prefix' is the fully-formed prefix, normally from compute_prefix above. -->
+    <xacro:macro name="rizon_srdf" params="prefix load_mounted_ft_sensor use_virtual_joint:=true">
         <group name="${prefix}arm">
             <chain base_link="${prefix}base_link" tip_link="${prefix}flange" />
