Commit message: feat: armN prefixes and per-arm initial positions on the dual branch
Two changes to the dual-arm (`Enlight-LL`, MICO) branch of
`flexiv_hardware/urdf/flexiv.urdf.xacro`.

**`armN` prefixes, forwarding `use_sn_prefix`.** Matches the description's
Enlight-LL branch, which now passes `arm1`/`arm2` and forwards the flag. The
two sides recompute the prefix independently, so both must agree or the
`ros2_control` block names joints the description never emitted and the
controller cannot claim its interfaces.

**Per-arm initial positions.** The branch hardcoded
`initial_positions_file_left="${arm_init}"`, ignoring the
`initial_positions_file` argument the single-arm branch honours. A dual robot
needs two poses and that argument names one file, so rather than overload it
this adds `initial_positions_file_left` / `initial_positions_file_right`.
Empty means "keep the vendor default for that arm", so callers that pass
neither behave exactly as before — which matters because this branch is
shared with the MICO models, whose right arm defaults to the mirrored file.

Without this a consumer cannot seed a simulated dual arm's start pose: the
mock hardware takes its initial values from the URDF, so the vendor default
was the only reachable pose.

Co-Authored-By: Claude Opus 5 (1M context) <noreply@anthropic.com>

File: flexiv_hardware/urdf/flexiv.urdf.xacro (robot description, xacro)
@@ -16,4 +16,11 @@
   <xacro:arg name="fake_sensor_commands" default="false" />
   <xacro:arg name="initial_positions_file" default="" />
+  <!--
+    Per-arm overrides for the dual-arm branch, which cannot use the single-arm
+    `initial_positions_file` above: that names one file and a dual robot needs
+    two. Empty means "keep the vendor default for that arm".
+  -->
+  <xacro:arg name="initial_positions_file_left" default="" />
+  <xacro:arg name="initial_positions_file_right" default="" />
   <!-- Robot model, including the arg declarations this file relies on
        (robot_sn, arm_prefix). -->
@@ -63,10 +70,17 @@
     <!-- ============ ONE ROBOT WITH TWO ARMS (Enlight-LL, MICO) ============ -->
     <xacro:if value="${is_enlight_ll or is_mico_core or is_mico_torso}">
-      <xacro:compute_arm_prefix arm_prefix="left" robot_sn="$(arg robot_sn)" />
+      <xacro:compute_arm_prefix arm_prefix="arm1" robot_sn="$(arg robot_sn)" use_sn_prefix="$(arg use_sn_prefix)" />
       <xacro:property name="prefix_left" value="${computed_arm_prefix}" lazy_eval="false" />
-      <xacro:compute_arm_prefix arm_prefix="right" robot_sn="$(arg robot_sn)" />
+      <xacro:compute_arm_prefix arm_prefix="arm2" robot_sn="$(arg robot_sn)" use_sn_prefix="$(arg use_sn_prefix)" />
       <xacro:property name="prefix_right" value="${computed_arm_prefix}" lazy_eval="false" />
       <!-- Enlight-LL mirrors nothing; the MICO arms face each other. -->
-      <xacro:property name="init_right" value="${arm_init if is_enlight_ll else arm_init_mirrored}" />
+      <xacro:property name="init_right_default"
+          value="${arm_init if is_enlight_ll else arm_init_mirrored}" />
+        <xacro:property name="init_left"
+          value="${'$(arg initial_positions_file_left)'
+                   if '$(arg initial_positions_file_left)' != '' else arm_init}" />
+        <xacro:property name="init_right"
+          value="${'$(arg initial_positions_file_right)'
+                   if '$(arg initial_positions_file_right)' != '' else init_right_default}" />
       <!-- MICO-Plus and MICO-Ultra add two actuated torso joints. -->
       <xacro:unless value="${is_mico_torso}">
@@ -78,5 +92,5 @@
           use_fake_hardware="$(arg use_fake_hardware)"
           fake_sensor_commands="$(arg fake_sensor_commands)"
-          initial_positions_file_left="${arm_init}"
+          initial_positions_file_left="${init_left}"
           initial_positions_file_right="${init_right}" />
       </xacro:unless>
@@ -89,5 +103,5 @@
           use_fake_hardware="$(arg use_fake_hardware)"
           fake_sensor_commands="$(arg fake_sensor_commands)"
-          initial_positions_file_left="${arm_init}"
+          initial_positions_file_left="${init_left}"
           initial_positions_file_right="${init_right}"
           torso_initial_positions_file="${cfg}/${rtype}/torso_initial_positions.yaml" />
